File: Hardware/badge/thirtyinone-badge.kicad_pcb (KiCad board)
At the start: 2 copper layers, 105 x 130 mm, 130 parts, among them J1 SWD, J105 Conn_01x02_Female, J106 Conn_01x02_Female, J107 Conn_01x02_Female, J108 Conn_01x02_Female, J109 Conn_01x02_Female, J110 Conn_01x02_Female, J111 Conn_01x02_Female, J112 Conn_01x02_Female, J113 Conn_01x02_Female, J114 Conn_01x02_Female, J115 Conn_01x02_Female, J116 Conn_01x02_Female, J117 Conn_01x02_Female, J118 Conn_01x02_Female, J119 Conn_01x02_Female, J120 Conn_01x02_Female, J121 Conn_01x02_Female, J122 Conn_01x02_Female, J123 Conn_01x02_Female, J124 Conn_01x02_Female, J125 Conn_01x02_Female, J126 Conn_01x02_Female, J127 Conn_01x02_Female, J128 Conn_01x02_Female, J129 Conn_01x02_Female, J130 Conn_01x02_Female, J131 Conn_01x02_Female, J132 Conn_01x02_Female, J133 Conn_01x02_Female, J134 Conn_01x02_Female, J135 Conn_01x02_Female, J136 Conn_01x02_Female, J137 Conn_01x02_Female, J138 Conn_01x02_Female, J139 Conn_01x02_Female, J140 Conn_01x02_Female, J141 Conn_01x02_Female, J142 Conn_01x02_Female, J143 Conn_01x02_Female, J144 Conn_01x02_Female, J145 Conn_01x02_Female, J146 Conn_01x02_Female, J147 Conn_01x02_Female, J148 Conn_01x02_Female, J149 Conn_01x02_Female, J150 Conn_01x02_Female, J151 Conn_01x02_Female, J152 Conn_01x02_Female, J153 Conn_01x02_Female, J154 Conn_01x02_Female, J155 Conn_01x02_Female, J156 Conn_01x02_Female, J157 Conn_01x02_Female, J158 Conn_01x02_Female, J159 Conn_01x03_Female, J160 Conn_01x03_Female, J161 Conn_01x03_Female, J162 Conn_01x03_Female, J163 Conn_01x03_Female, J164 Conn_01x03_Female, J165 Conn_01x03_Female, J166 Conn_01x03_Female, J167 Conn_01x03_Female, J168 Conn_01x02_Female, J169 Conn_01x02_Female, J170 Battery +, J171 Battery -, J172 Spare, J173 Spare, J174 Spare, J175 Spare, J2 TagConnect, J3 OLED, J4 USB3140-30-0170-1-C, J5 uC Interface, Q101 3904, Q102 3904, Q103 3906, SW1 Power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

Commit message: Updated to hardware version 1.1 to reflect some footprint fixes, and swap to an alternate microcontroller due to parts availability
Parts:
- removed C6: 0.1uF, Capacitor_SMD:C_0603_1608Metric
- added G***: LOGO, lib_fp:BackSilk-Text, B.Cu at (135.5, 85.8)
- BOOT1: footprint Button_Switch_SMD:SW_Push_1P1T_NO_6x6mm_H9.5mm -> lib_fp:SW_Push_1P1T_NO_CK_PTS526
- D3, D4: footprint Package_TO_SOT_SMD:SOT-323_SC-70 -> Package_TO_SOT_SMD:SOT-23
- U2: value ATSAMD21G15A-A -> ATSAMD21E15B-AU; footprint Package_QFP:TQFP-48_7x7mm_P0.5mm -> Package_QFP:TQFP-32_7x7mm_P0.8mm
- moved C4 3.89 mm to (101.7, 33.0)
- moved C5 3.89 mm to (103.2, 33.0)
- moved D3 1.20 mm to (122.9, 31.8)
- moved C9 0.82 mm to (92.4, 29.1)
- moved C10 0.82 mm to (92.4, 35.2)
- moved R1 0.82 mm to (93.1, 31.3)
- moved R2 0.82 mm to (93.1, 32.9)
- moved J4 0.81 mm to (88.5, 31.8)
- moved D4 0.47 mm to (119.3, 31.8)
Connections:
- D4 pad 3: ADC2 -> ADC0
- J5 pad 9: ADC2 -> ADC0
- U2 pad 10: PWM1 -> GND
- U2 pad 11: unconnected-(U2-Pad11) -> SDA
- U2 pad 12: unconnected-(U2-Pad12) -> SCL
- U2 pad 13: SDA -> PWM0
- U2 pad 14: SCL -> PWM1
- U2 pad 16: unconnected-(U2-Pad16) -> Net-(BOOT1-Pad2)
- U2 pad 17: +3V3 -> GPIO0
- U2 pad 18: GND -> GPIO1
- U2 pad 19: unconnected-(U2-Pad19) -> GPIO2
- U2 pad 20: unconnected-(U2-Pad20) -> GPIO3
- U2 pad 23: unconnected-(U2-Pad23) -> USB_N
- U2 pad 24: Net-(BOOT1-Pad2) -> USB_P
- U2 pad 26: unconnected-(U2-Pad26) -> RESET
- U2 pad 27: GPIO0 -> unconnected-(U2-Pad27)
- U2 pad 28: GPIO1 -> GND
- U2 pad 29: GPIO2 -> Net-(C8-Pad1)
- U2 pad 30: GPIO3 -> +3V3
- U2 pad 31: unconnected-(U2-Pad31) -> SWCLK
- U2 pad 32: unconnected-(U2-Pad32) -> SWDIO
- U2 pad 4: unconnected-(U2-Pad4) -> ADC1
- U2 pad 5: GND -> ADC0
- U2 pad 6: +3V3 -> unconnected-(U2-Pad6)
- U2 pad 7: ADC1 -> unconnected-(U2-Pad7)
- U2 pad 8: ADC2 -> unconnected-(U2-Pad8)
- U2 pad 9: PWM0 -> +3V3
Routing:
- net ADC2: track 24.1 -> 0.00 mm, vias 2 -> 0
- net ADC0: track 0.00 -> 21.8 mm, vias 0 -> 2
- net GND: track 76.5 -> 58.2 mm
- net +3V3: track 240.8 -> 230.4 mm
- net PWM2: track 5.56 -> 9.73 mm
- net USB_P: track 37.4 -> 40.1 mm
- net PWM1: track 8.83 -> 11.4 mm
- net USB_N: track 40.6 -> 43.0 mm
- net Net-(BOOT1-Pad2): track 39.4 -> 37.2 mm, vias 0 -> 2
- net RESET: track 41.3 -> 39.2 mm
- net SCL: track 16.5 -> 14.6 mm
- net DAC0: track 16.8 -> 15.0 mm
- net RX: track 25.7 -> 24.1 mm
- net PWM0: track 11.5 -> 13.0 mm
- net TX: track 25.4 -> 24.0 mm
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Other:
- board text added: "ADC0"
- board text removed: "ADC2"
